Commit message: gazebo working

File: urdf/yantra_robot.urdf.xacro (robot description, xacro)
@@ -55,8 +55,8 @@
 		</link>
 		<gazebo reference="link_${i}">
-			<!--mu1 value="200.0"/>
-			<mu2 value="100.0"/>
-			<kp value="100000.0"/>
-			<kd value="1"/-->
+			<mu1 value="30.0"/>
+			<mu2 value="30.0"/>
+			<kp value="1000000.0"/>
+			<kd value="100.0"/>
 			<material>Gazebo/BlackTransparent</material>
 		</gazebo>
@@ -85,8 +85,8 @@
 			<actuator name="actuator_${i}_${j}">
 				<mechanicalReduction>1</mechanicalReduction>
-				<hardwareInterface>hardware_interface/VelocityJointInterface</hardwareInterface>
+				<hardwareInterface>hardware_interface/PositionJointInterface</hardwareInterface>
 			</actuator>
-			<joint name="link_${i}_${j}">
-				<hardwareInterface>hardware_interface/VelocityJointInterface</hardwareInterface>
+			<joint name="joint_${i}_${j}">
+				<hardwareInterface>hardware_interface/PositionJointInterface</hardwareInterface>
 			</joint>
 		</transmission>
@@ -110,4 +110,9 @@
 		<material>Gazebo/BlackTransparent</material>
 	</gazebo-->
+	<link name="world"/>
+	<joint name="world_link_0" type="fixed">
+		<parent link="world"/>
+		<child link="link_0"/>
+	</joint>
 	<xacro:link i="0" r="0" p="0" x="0" y="0" z="${h0/2}" m="${m0}" rad="${r0}" ht="${h0}" rot_axis="z"/>
 	<xacro:link i="1" r="0" p="0" x="0" y="0" z="${h1/2}" m="${m1}" rad="${r1}" ht="${h1}" rot_axis="z"/>
@@ -130,5 +135,5 @@
 	<gazebo>
 		<plugin name="gazebo_ros_control" filename="libgazebo_ros_control.so">
-			<robotNamespace>/</robotNamespace>
+			<robotNamespace>/yantra</robotNamespace>
 		</plugin>
 	</gazebo>

Commit message: PID tuned(not finely tuned)

File: urdf/yantra_robot.urdf.xacro (robot description, xacro)
@@ -44,5 +44,5 @@
 				<mass value="${m}"/>
 				<xacro:if value="${rot_axis == 'x'}">
-					<inertia ixx="${m*ht*ht/3}" ixy="0" ixz="0" iyy="0" iyz="0" izz="${m*ht*ht/3}"/>
+					<inertia iyy="${m*ht*ht/3}" ixy="0" ixz="0" ixx="0" iyz="0" izz="${m*ht*ht/3}"/>
 				</xacro:if>
 				<xacro:if value="${rot_axis == 'z'}">
@@ -76,17 +76,17 @@
 			<origin xyz="${x} ${y} ${z}" rpy="${rr} ${pp} ${yy}"/>
 			<axis xyz="${rx} ${ry} ${rz}"/>
-			<limit effort="1" upper="3.124" lower="-3.124" velocity="2.094"/>
+			<limit effort="1000000" upper="3.3" lower="-3.3" velocity="200000"/>
 		</joint>
 		</xacro:if>
 	</xacro:macro>
-	<xacro:macro name="joint_transmission" params="i j">
+	<xacro:macro name="joint_transmission" params="i j r">
 		<transmission name="transmission_${i}_${j}">
 			<type>transmission_interface/SimpleTransmission</type>
 			<actuator name="actuator_${i}_${j}">
 				<mechanicalReduction>1</mechanicalReduction>
-				<hardwareInterface>hardware_interface/PositionJointInterface</hardwareInterface>
+				<hardwareInterface>EffortJointInterface</hardwareInterface>
 			</actuator>
 			<joint name="joint_${i}_${j}">
-				<hardwareInterface>hardware_interface/PositionJointInterface</hardwareInterface>
+					<hardwareInterface>hardware_interface/EffortJointInterface</hardwareInterface>
 			</joint>
 		</transmission>
@@ -128,9 +128,9 @@
 	<xacro:link_joints plink="4" clink="51" x="0" y="0" z="${h4}" rr="0" pp="0" yy="0" jtype="r" rx="0" ry="1" rz="0"/>
 	<xacro:link_joints plink="51" clink="52" x="0" y="0" z="${h51}" rr="0" pp="0" yy="0" jtype="f" rx="0" ry="0" rz="0"/>
-	<xacro:joint_transmission i="0" j="1"/>
-	<xacro:joint_transmission i="1" j="2"/>
-	<xacro:joint_transmission i="2" j="3"/>
-	<xacro:joint_transmission i="3" j="4"/>
-	<xacro:joint_transmission i="4" j="51"/>
+	<xacro:joint_transmission i="0" j="1" r="1"/>
+	<xacro:joint_transmission i="1" j="2" r="50"/>
+	<xacro:joint_transmission i="2" j="3" r="50"/>
+	<xacro:joint_transmission i="3" j="4" r="50"/>
+	<xacro:joint_transmission i="4" j="51" r="50"/>
 	<gazebo>
 		<plugin name="gazebo_ros_control" filename="libgazebo_ros_control.so">

Commit message: publish commands done

File: urdf/yantra_robot.urdf.xacro (robot description, xacro)
@@ -62,5 +62,5 @@
 		</gazebo>
 	</xacro:macro>
-	<xacro:macro name="link_joints" params="plink clink jtype x y z rx ry rz rr pp yy">
+	<xacro:macro name="link_joints" params="plink clink jtype x y z rx ry rz rr pp yy efrt">
 		<xacro:if value="${jtype == 'f'}">
 		<joint name="joint_${plink}_${clink}" type="fixed">
@@ -76,9 +76,9 @@
 			<origin xyz="${x} ${y} ${z}" rpy="${rr} ${pp} ${yy}"/>
 			<axis xyz="${rx} ${ry} ${rz}"/>
-			<limit effort="1000000" upper="3.3" lower="-3.3" velocity="200000"/>
+			<limit effort="${efrt}" upper="3.3" lower="-3.3" velocity="200000"/>
 		</joint>
 		</xacro:if>
 	</xacro:macro>
-	<xacro:macro name="joint_transmission" params="i j r">
+	<xacro:macro name="joint_transmission" params="i j">
 		<transmission name="transmission_${i}_${j}">
 			<type>transmission_interface/SimpleTransmission</type>
@@ -122,15 +122,15 @@
 	<xacro:link i="51" r="0" p="0" x="0" y="0" z="${h51/2}" m="${m51}" rad="${r51}" ht="${h51}" rot_axis="x"/>
 	<xacro:link i="52" r="0" p="${pi/2}" x="${h52/2 - r51}" y="0" z="0" m="${m52}" rad="${r52}" ht="${h52}" rot_axis="n"/>
-	<xacro:link_joints plink="0" clink="1" x="0" y="0" z="${h0}" rr="0" pp="0" yy="0" jtype="r" rx="0" ry="0" rz="1"/>
-	<xacro:link_joints plink="1" clink="2" x="0" y="0" z="${h1}" rr="0" pp="0" yy="0" jtype="r" rx="0" ry="1" rz="0"/>
-	<xacro:link_joints plink="2" clink="3" x="0" y="0" z="${h2}" rr="0" pp="0" yy="0" jtype="r" rx="0" ry="1" rz="0"/>
-	<xacro:link_joints plink="3" clink="4" x="0" y="0" z="${h3}" rr="0" pp="0" yy="0" jtype="r" rx="0" ry="0" rz="1"/>
-	<xacro:link_joints plink="4" clink="51" x="0" y="0" z="${h4}" rr="0" pp="0" yy="0" jtype="r" rx="0" ry="1" rz="0"/>
-	<xacro:link_joints plink="51" clink="52" x="0" y="0" z="${h51}" rr="0" pp="0" yy="0" jtype="f" rx="0" ry="0" rz="0"/>
-	<xacro:joint_transmission i="0" j="1" r="1"/>
-	<xacro:joint_transmission i="1" j="2" r="50"/>
-	<xacro:joint_transmission i="2" j="3" r="50"/>
-	<xacro:joint_transmission i="3" j="4" r="50"/>
-	<xacro:joint_transmission i="4" j="51" r="50"/>
+	<xacro:link_joints plink="0" clink="1" x="0" y="0" z="${h0}" rr="0" pp="0" yy="0" jtype="r" rx="0" ry="0" rz="1" efrt="10"/>
+	<xacro:link_joints plink="1" clink="2" x="0" y="0" z="${h1}" rr="0" pp="0" yy="0" jtype="r" rx="0" ry="1" rz="0" efrt="500"/>
+	<xacro:link_joints plink="2" clink="3" x="0" y="0" z="${h2}" rr="0" pp="0" yy="0" jtype="r" rx="0" ry="1" rz="0" efrt="300"/>
+	<xacro:link_joints plink="3" clink="4" x="0" y="0" z="${h3}" rr="0" pp="0" yy="0" jtype="r" rx="0" ry="0" rz="1" efrt="10"/>
+	<xacro:link_joints plink="4" clink="51" x="0" y="0" z="${h4}" rr="0" pp="0" yy="0" jtype="r" rx="0" ry="1" rz="0" efrt="10"/>
+	<xacro:link_joints plink="51" clink="52" x="0" y="0" z="${h51}" rr="0" pp="0" yy="0" jtype="f" rx="0" ry="0" rz="0" efrt="10"/>
+	<xacro:joint_transmission i="0" j="1"/>
+	<xacro:joint_transmission i="1" j="2"/>
+	<xacro:joint_transmission i="2" j="3"/>
+	<xacro:joint_transmission i="3" j="4"/>
+	<xacro:joint_transmission i="4" j="51"/>
 	<gazebo>
 		<plugin name="gazebo_ros_control" filename="libgazebo_ros_control.so">

Commit message: controller set. But not useful. falls at init

File: urdf/yantra_robot.urdf.xacro (robot description, xacro)
@@ -71,10 +71,11 @@
 		</xacro:if>
 		<xacro:if value="${jtype == 'r'}">
-		<joint name="joint_${plink}_${clink}" type="revolute">
+		<!--joint name="joint_${plink}_${clink}" type="revolute"-->
+		<joint name="joint_${plink}_${clink}" type="continuous">
 			<parent link="link_${plink}"/>
 			<child link="link_${clink}"/>
 			<origin xyz="${x} ${y} ${z}" rpy="${rr} ${pp} ${yy}"/>
 			<axis xyz="${rx} ${ry} ${rz}"/>
-			<limit effort="${efrt}" upper="3.3" lower="-3.3" velocity="200000"/>
+			<limit effort="${efrt}"  upper="100" lower="100" velocity="20"/>
 		</joint>
 		</xacro:if>
@@ -85,5 +86,4 @@
 			<actuator name="actuator_${i}_${j}">
 				<mechanicalReduction>1</mechanicalReduction>
-				<hardwareInterface>VelocityJointInterface</hardwareInterface>
 			</actuator>
 			<joint name="joint_${i}_${j}">

Commit message: switching to controller_swtiching branch

File: urdf/yantra_robot.urdf.xacro (robot description, xacro)
@@ -77,5 +77,5 @@
 			<origin xyz="${x} ${y} ${z}" rpy="${rr} ${pp} ${yy}"/>
 			<axis xyz="${rx} ${ry} ${rz}"/>
-			<limit effort="${efrt}"  upper="100" lower="100" velocity="20"/>
+			<limit effort="${efrt}"  upper="100" lower="100" velocity="2000"/>
 		</joint>
 		</xacro:if>
@@ -88,5 +88,5 @@
 			</actuator>
 			<joint name="joint_${i}_${j}">
-					<hardwareInterface>hardware_interface/VelocityJointInterface</hardwareInterface>
+					<hardwareInterface>hardware_interface/EffortJointInterface</hardwareInterface>
 			</joint>
 		</transmission>

Commit message: DH parameter verified

File: urdf/yantra_robot.urdf.xacro (robot description, xacro)
@@ -21,5 +21,5 @@
 	<xacro:property name="h4" value="0.167"/>
 	<xacro:property name="h51" value="0.112"/>
-	<xacro:property name="h52" value="0.104"/>
+	<xacro:property name="h52" value="0.116"/>
 	<material name="red_trans">
 		<color rgba="1 0 0 0.5"/>
@@ -121,7 +121,5 @@
 	<xacro:link i="4" r="0" p="0" x="0" y="0" z="${h4/2}" m="${m4}" rad="${r4}" ht="${h4}" rot_axis="z"/>
 	<xacro:link i="51" r="0" p="0" x="0" y="0" z="${h51/2}" m="${m51}" rad="${r51}" ht="${h51}" rot_axis="x"/>
-	<!--
 	<xacro:link i="52" r="0" p="${pi/2}" x="${h52/2 - r51}" y="0" z="0" m="${m52}" rad="${r52}" ht="${h52}" rot_axis="n"/>
-	-->
 	<xacro:link_joints plink="0" clink="1" x="0" y="0" z="${h0}" rr="0" pp="0" yy="0" jtype="r" rx="0" ry="0" rz="1" efrt="10"/>
 	<xacro:link_joints plink="1" clink="2" x="0" y="0" z="${h1}" rr="0" pp="0" yy="0" jtype="r" rx="0" ry="1" rz="0" efrt="500"/>
@@ -129,7 +127,5 @@
 	<xacro:link_joints plink="3" clink="4" x="0" y="0" z="${h3}" rr="0" pp="0" yy="0" jtype="r" rx="0" ry="0" rz="1" efrt="10"/>
 	<xacro:link_joints plink="4" clink="51" x="0" y="0" z="${h4}" rr="0" pp="0" yy="0" jtype="r" rx="0" ry="1" rz="0" efrt="10"/>
-	<!--
 	<xacro:link_joints plink="51" clink="52" x="0" y="0" z="${h51}" rr="0" pp="0" yy="0" jtype="f" rx="0" ry="0" rz="0" efrt="10"/>
-	-->
 	<xacro:joint_transmission i="0" j="1"/>
 	<xacro:joint_transmission i="1" j="2"/>

Commit message: complete except seg fault

File: urdf/yantra_robot.urdf.xacro (robot description, xacro)
@@ -111,4 +111,5 @@
 	</gazebo-->
 	<link name="world"/>
+	<link name="tcp"/>
 	<joint name="world_link_0" type="fixed">
 		<parent link="world"/>
@@ -117,15 +118,15 @@
 	<xacro:link i="0" r="0" p="0" x="0" y="0" z="${h0/2}" m="${m0}" rad="${r0}" ht="${h0}" rot_axis="z"/>
 	<xacro:link i="1" r="0" p="0" x="0" y="0" z="${h1/2}" m="${m1}" rad="${r1}" ht="${h1}" rot_axis="z"/>
-	<xacro:link i="2" r="0" p="0" x="0" y="0" z="${h2/2}" m="${m2}" rad="${r2}" ht="${h2}" rot_axis="x"/>
-	<xacro:link i="3" r="0" p="0" x="0" y="0" z="${h3/2}" m="${m3}" rad="${r3}" ht="${h3}" rot_axis="x"/>
+	<xacro:link i="2" r="${-pi/2}" p="0" x="0" y="${h2/2}" z="0" m="${m2}" rad="${r2}" ht="${h2}" rot_axis="x"/>
+	<xacro:link i="3" r="0" p="${pi/2}" x="${h3/2}" y="0" z="0" m="${m3}" rad="${r3}" ht="${h3}" rot_axis="x"/>
 	<xacro:link i="4" r="0" p="0" x="0" y="0" z="${h4/2}" m="${m4}" rad="${r4}" ht="${h4}" rot_axis="z"/>
-	<xacro:link i="51" r="0" p="0" x="0" y="0" z="${h51/2}" m="${m51}" rad="${r51}" ht="${h51}" rot_axis="x"/>
-	<xacro:link i="52" r="0" p="${pi/2}" x="${h52/2 - r51}" y="0" z="0" m="${m52}" rad="${r52}" ht="${h52}" rot_axis="n"/>
+	<xacro:link i="51" r="0" p="${pi/2}" x="${-h51/2}" y="0" z="0" m="${m51}" rad="${r51}" ht="${h51}" rot_axis="x"/>
+	<xacro:link i="52" r="${pi/2}" p="0" y="${h52/2 - r51}" x="0" z="0" m="${m52}" rad="${r52}" ht="${h52}" rot_axis="n"/>
 	<xacro:link_joints plink="0" clink="1" x="0" y="0" z="${h0}" rr="0" pp="0" yy="0" jtype="r" rx="0" ry="0" rz="1" efrt="10"/>
-	<xacro:link_joints plink="1" clink="2" x="0" y="0" z="${h1}" rr="0" pp="0" yy="0" jtype="r" rx="0" ry="1" rz="0" efrt="500"/>
-	<xacro:link_joints plink="2" clink="3" x="0" y="0" z="${h2}" rr="0" pp="0" yy="0" jtype="r" rx="0" ry="1" rz="0" efrt="300"/>
-	<xacro:link_joints plink="3" clink="4" x="0" y="0" z="${h3}" rr="0" pp="0" yy="0" jtype="r" rx="0" ry="0" rz="1" efrt="10"/>
-	<xacro:link_joints plink="4" clink="51" x="0" y="0" z="${h4}" rr="0" pp="0" yy="0" jtype="r" rx="0" ry="1" rz="0" efrt="10"/>
-	<xacro:link_joints plink="51" clink="52" x="0" y="0" z="${h51}" rr="0" pp="0" yy="0" jtype="f" rx="0" ry="0" rz="0" efrt="10"/>
+	<xacro:link_joints plink="1" clink="2" x="0" y="0" z="${h1}" rr="${pi/2}" pp="0" yy="0" jtype="r" rx="0" ry="0" rz="1" efrt="500"/>
+	<xacro:link_joints plink="2" clink="3" x="0" y="${h2}" z="0" rr="0" pp="0" yy="${pi/2}" jtype="r" rx="0" ry="0" rz="1" efrt="300"/>
+	<xacro:link_joints plink="3" clink="4" x="${h3}" y="0" z="0" rr="${pi/2}" pp="0" yy="${pi/2}" jtype="r" rx="0" ry="0" rz="1" efrt="10"/>
+	<xacro:link_joints plink="4" clink="51" x="0" y="0" z="${h4}" rr="${pi/2}" pp="0" yy="${pi}" jtype="r" rx="0" ry="0" rz="1" efrt="10"/>
+	<xacro:link_joints plink="51" clink="52" x="${-h51}" y="0" z="0" rr="0" pp="0" yy="0" jtype="f" rx="0" ry="0" rz="0" efrt="10"/>
 	<xacro:joint_transmission i="0" j="1"/>
 	<xacro:joint_transmission i="1" j="2"/>
@@ -133,4 +134,9 @@
 	<xacro:joint_transmission i="3" j="4"/>
 	<xacro:joint_transmission i="4" j="51"/>
+	<joint name="tcp_joint" type="fixed">
+		<parent link="link_52"/>
+		<child link="tcp"/>
+		<origin xyz="0 0 0" rpy="0 0 0"/>
+	</joint>
 	<gazebo>
 		<plugin name="gazebo_ros_control" filename="libgazebo_ros_control.so">

Commit message: initial commit

File: urdf/yantra_robot.urdf.xacro (robot description, xacro)
@@ -77,5 +77,5 @@
 			<origin xyz="${x} ${y} ${z}" rpy="${rr} ${pp} ${yy}"/>
 			<axis xyz="${rx} ${ry} ${rz}"/>
-			<limit effort="${efrt}"  upper="100" lower="100" velocity="2000"/>
+			<limit effort="${efrt}"  upper="100" lower="100" velocity="20000000"/>
 		</joint>
 		</xacro:if>
@@ -123,5 +123,5 @@
 	<xacro:link i="51" r="0" p="${pi/2}" x="${-h51/2}" y="0" z="0" m="${m51}" rad="${r51}" ht="${h51}" rot_axis="x"/>
 	<xacro:link i="52" r="${pi/2}" p="0" y="${h52/2 - r51}" x="0" z="0" m="${m52}" rad="${r52}" ht="${h52}" rot_axis="n"/>
-	<xacro:link_joints plink="0" clink="1" x="0" y="0" z="${h0}" rr="0" pp="0" yy="0" jtype="r" rx="0" ry="0" rz="1" efrt="10"/>
+	<xacro:link_joints plink="0" clink="1" x="0" y="0" z="${h0}" rr="0" pp="0" yy="0" jtype="r" rx="0" ry="0" rz="1" efrt="100"/>
 	<xacro:link_joints plink="1" clink="2" x="0" y="0" z="${h1}" rr="${pi/2}" pp="0" yy="0" jtype="r" rx="0" ry="0" rz="1" efrt="500"/>
 	<xacro:link_joints plink="2" clink="3" x="0" y="${h2}" z="0" rr="0" pp="0" yy="${pi/2}" jtype="r" rx="0" ry="0" rz="1" efrt="300"/>
